Commit message: Final update

File: urdf/yaskawa_wth_gripper.xacro (robot description, xacro)
@@ -12,5 +12,6 @@
 	<xacro:include filename="$(find realsense2_description)/urdf/_d435i.urdf.xacro"/>
 	<xacro:sensor_d435i parent="base_link_gripper">
-		<origin xyz="-0.032192 0.021689 0.095" rpy="0 ${25*deg} ${-90*deg}" />
+		<origin xyz="-0.032192 0.021689 0.095" rpy="0 ${21.5*deg} ${-90*deg}" />
+		<!-- <origin xyz="-0.032192 0.021689 0.095" rpy="0 ${25*deg} ${-90*deg}" /> -->
 	</xacro:sensor_d435i>
 	<!-- end effector frame -->

Commit message: Fix

File: urdf/yaskawa_wth_gripper.xacro (robot description, xacro)
@@ -12,11 +12,11 @@
 	<xacro:include filename="$(find realsense2_description)/urdf/_d435i.urdf.xacro"/>
 	<xacro:sensor_d435i parent="base_link_gripper">
-		<origin xyz="-0.032192 0.021689 0.095" rpy="0 ${21.5*deg} ${-90*deg}" />
-		<!-- <origin xyz="-0.032192 0.021689 0.095" rpy="0 ${25*deg} ${-90*deg}" /> -->
+		<origin xyz="-0.034192 0.021689 0.095" rpy="0 ${21.7*deg} ${-90*deg}" />
+		<!-- <origin xyz="-0.032192 0.021689 0.095" rpy="0 ${21.5*deg} ${-90*deg}" /> -->
 	</xacro:sensor_d435i>
 	<!-- end effector frame -->
 	<link name="end_effector_tool0" />
 	<joint name="tool0-end_effector_tool0" type="fixed" >
-		<origin xyz="0 0 0.21" rpy="0 0 0"/>
+		<origin xyz="0 0.0055 0.21" rpy="0 0 0"/>
 		<parent link="tool0" />
 		<child link="end_effector_tool0" />

Commit message: Add place with optimization

File: urdf/yaskawa_wth_gripper.xacro (robot description, xacro)
@@ -18,5 +18,5 @@
 	<link name="end_effector_tool0" />
 	<joint name="tool0-end_effector_tool0" type="fixed" >
-		<origin xyz="0 0.0055 0.21" rpy="0 0 0"/>
+		<origin xyz="0 0.0075 0.21" rpy="0 0 0"/>
 		<parent link="tool0" />
 		<child link="end_effector_tool0" />

File: urdf/yaskawa_wth_gripper_30_96.xacro (robot description, xacro)
@@ -12,5 +12,7 @@
 	<xacro:include filename="$(find realsense2_description)/urdf/_d435i.urdf.xacro"/>
 	<xacro:sensor_d435i parent="base_link_gripper">
-		<origin xyz="-0.001 -0.004 0.126" rpy="${0*deg}  ${20.7*deg} ${-91*deg}" />
+		<origin xyz="-0.0005 -0.004 0.126" rpy="${0*deg}  ${21.2*deg} ${-91*deg}" />
+		<!-- <origin xyz="-0.001 -0.004 0.126" rpy="${0*deg}  ${21.2*deg} ${-91*deg}" /> BUONO -->
+		<!-- <origin xyz="-0.001 -0.004 0.126" rpy="${0*deg}  ${20.7*deg} ${-91*deg}" /> -->
 		<!-- <origin xyz="-0.032192 0.021689 0.095" rpy="0 ${21.5*deg} ${-90*deg}" /> -->
 	</xacro:sensor_d435i>
@@ -18,5 +20,6 @@
 	<link name="end_effector_tool0" />
 	<joint name="tool0-end_effector_tool0" type="fixed" >
-		<origin xyz="0 0.0 0.21" rpy="0 0 0"/>
+		<!-- <origin xyz="0 0.0065 0.21" rpy="0 0 0"/> -->
+		<origin xyz="0 0.007 0.21" rpy="0 0 0"/>
 		<parent link="tool0" />
 		<child link="end_effector_tool0" />
@@ -25,5 +28,5 @@
 	<link name="push_frame" />
 	<joint name="push_joint" type="fixed" >
-		<origin xyz="0.0235 -0.0673 0.036" rpy="0 0 0"/>
+		<origin xyz="0.0325 -0.074 0.033" rpy="0 0 0"/>
 		<parent link="push_extension" />
 		<child link="push_frame" />
