Commit message: add_push

File: urdf/yaskawa_wth_gripper_30_96.xacro (robot description, xacro)
@@ -22,3 +22,10 @@
 		<child link="end_effector_tool0" />
 	</joint>
+	<!-- push frame -->
+	<link name="push_frame" />
+	<joint name="push_joint" type="fixed" >
+		<origin xyz="0.0235 -0.0673 0.036" rpy="0 0 0"/>
+		<parent link="push_extension" />
+		<child link="push_frame" />
+	</joint>
 </robot>

Commit message: Fixed planning server to grasp

File: urdf/yaskawa_wth_gripper_30_96.xacro (robot description, xacro)
@@ -21,5 +21,5 @@
 	<joint name="tool0-end_effector_tool0" type="fixed" >
 		<!-- <origin xyz="0 0.0065 0.21" rpy="0 0 0"/> -->
-		<origin xyz="0 0.007 0.21" rpy="0 0 0"/>
+		<origin xyz="0 0.0 0.21" rpy="0 0 0"/>
 		<parent link="tool0" />
 		<child link="end_effector_tool0" />

Commit message: Fixed apple gras p

File: urdf/yaskawa_wth_gripper_30_96.xacro (robot description, xacro)
@@ -21,5 +21,5 @@
 	<joint name="tool0-end_effector_tool0" type="fixed" >
 		<!-- <origin xyz="0 0.0065 0.21" rpy="0 0 0"/> -->
-		<origin xyz="0 0.0 0.21" rpy="0 0 0"/>
+		<origin xyz="0 0.01 0.21" rpy="0 0 0"/>
 		<parent link="tool0" />
 		<child link="end_effector_tool0" />
